File: antmicro-hdmi-mipi-bridge-hw.kicad_sch (KiCad schematic)
At the start: 0 parts

Commit message: Introduce component standardization
Other:
- title: Antmicro HDMI MIPI Bridge -> HDMI-MIPI Bridge
