File: csi.kicad_sch (KiCad schematic)
At the start: 5 parts, among them J6 Conn_FFC_WE_68715014022

Commit message: [#58304] Fix schematic after components lib rebase
Parts:
- SP1, SP2, SP3, SP4: Public (none) -> False
Changed lines of the file:
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@@
       (effects (font (size 1.27 1.27) (thickness 0.15)) (justify left bottom) hide)
+    )
+    (property "Public" "False" (at 396.24 251.46 0)
+      (effects (font (size 1.27 1.27)) (justify left bottom) hide)
     )
     (pin "1")
@@
       (effects (font (size 1.27 1.27) (thickness 0.15)) (justify left bottom) hide)
     )
+    (property "Public" "False" (at 368.3 238.76 0)
+      (effects (font (size 1.27 1.27)) (justify left bottom) hide)
+    )
     (pin "1")
     (instances
@@
     (property "License" "Apache-2.0" (at 396.24 246.38 0)
       (effects (font (size 1.27 1.27) (thickness 0.15)) (justify left bottom) hide)
+    )
+    (property "Public" "False" (at 396.24 238.76 0)
+      (effects (font (size 1.27 1.27)) (justify left bottom) hide)
     )
     (pin "1")
@@
       (effects (font (size 1.27 1.27) (thickness 0.15)) (justify left bottom) hide)
     )
+    (property "Public" "False" (at 368.3 251.46 0)
+      (effects (font (size 1.27 1.27)) (justify left bottom) hide)
+    )
     (pin "1")
